File: hardware/MainPCB/MainPCB.kicad_pcb (KiCad board)
At the start: 2 copper layers, 105.5 x 50 mm, 53 parts, among them J1 Conn_01x05, J2 Conn_01x02, J3 Conn_01x03, J4 USB4125-GF-A_REVA2, Q1 TIP120, SW2 SW_Push, U1 ESP32-CAM, U2 RASPBERRY_PI_PICO, U3 LSM6DSO32XTR

Commit message: feat: oh yea we need gerbers
Routing:
- net GND_LED: vias 3 -> 0
- net GND: vias 10 -> 2
Other:
- board text added: "cut along this line to seperate into 2 pcbs"
Changed lines of the file:
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@@
 		(tags "solder jumper open")
 		(property "Reference" "JP1"
-			(at -1.75 -2.5 180)
+			(at -0.5 -2.5 180)
 			(layer "F.SilkS")
 			(effects
@@
 		)
 		(fp_text user "3"
-			(at 1 2 90)
+			(at 1 2 180)
 			(layer "F.SilkS")
 			(effects
@@
 		)
 		(fp_text user "1"
-			(at -1.5 2 90)
+			(at -1.5 2 180)
 			(layer "F.SilkS")
 			(effects
@@
 		(tags "resistor")
 		(property "Reference" "R1"
-			(at -0.75 2 180)
+			(at 0 2 180)
 			(layer "F.SilkS")
 			(effects
@@
 	)
 	(gr_text "ECSE Design Competition 2026 - Part 2 Team 2:\nPhoenix, Siddhesh, Connor, Gao, Leon, Lauren, David"
-		(at 61.5 53.5 0)
+		(at 62 53.5 0)
 		(layer "F.SilkS")
 		(effects
@@
 		)
 	)
+	(gr_text "cut along this line to seperate into 2 pcbs"
+		(at 102 85.5 0)
+		(layer "B.SilkS")
+		(effects
+			(font
+				(size 0.8 0.8)
+				(thickness 0.2)
+				(bold yes)
+			)
+			(justify mirror)
+		)
+	)
 	(gr_text "VLED"
 		(at 73.3 92.7 0)
@@
 		(net "GND_LED")
 	)
-	(via
-		(at 120 90)
-		(size 0.6)
-		(drill 0.3)
-		(layers "F.Cu" "B.Cu")
-		(net "GND_LED")
-	)
-	(via
-		(at 140 90)
-		(size 0.6)
-		(drill 0.3)
-		(layers "F.Cu" "B.Cu")
-		(net "GND_LED")
-	)
-	(via
-		(at 130 90)
-		(size 0.6)
-		(drill 0.3)
-		(layers "F.Cu" "B.Cu")
-		(net "GND_LED")
-	)
 	(segment
 		(start 69 68.5)
@@
 	)
 	(segment
-		(start 72 67)
-		(end 72 66.75)
+		(start 72.75 67.75)
+		(end 70.8125 65.8125)
 		(width 0.25)
 		(layer "F.Cu")
@@
 	)
 	(segment
-		(start 71.0625 65.8125)
+		(start 70.8125 65.8125)
 		(end 68.5622 65.8125)
 		(width 0.25)
@@
 	)
 	(segment
-		(start 72 66.75)
-		(end 71.0625 65.8125)
-		(width 0.25)
-		(layer "F.Cu")
-		(net "/MISO")
-	)
-	(segment
-		(start 72.75 67.75)
-		(end 72 67)
+		(start 72.75 68.25)
+		(end 72.75 67.75)
 		(width 0.25)
 		(layer "F.Cu")
@@
 	)
 	(segment
-		(start 72.75 68.25)
-		(end 72.75 67.75)
-		(width 0.25)
-		(layer "F.Cu")
-		(net "/MISO")
-	)
-	(segment
 		(start 73.25 72.5)
 		(end 72.22 73.53)
@@
 	)
 	(via
-		(at 150 70)
-		(size 0.6)
-		(drill 0.3)
-		(layers "F.Cu" "B.Cu")
-		(net "GND")
-	)
-	(via
-		(at 130 60)
-		(size 0.6)
-		(drill 0.3)
-		(layers "F.Cu" "B.Cu")
-		(net "GND")
-	)
-	(via
-		(at 140 60)
-		(size 0.6)
-		(drill 0.3)
-		(layers "F.Cu" "B.Cu")
-		(net "GND")
-	)
-	(via
-		(at 140 70)
-		(size 0.6)
-		(drill 0.3)
-		(layers "F.Cu" "B.Cu")
-		(net "GND")
-	)
-	(via
-		(at 80 60)
-		(size 0.6)
-		(drill 0.3)
-		(layers "F.Cu" "B.Cu")
-		(net "GND")
-	)
-	(via
-		(at 120 60)
-		(size 0.6)
-		(drill 0.3)
-		(layers "F.Cu" "B.Cu")
-		(net "GND")
-	)
-	(via
 		(at 63.5 62)
 		(size 0.6)
@@
 		(net "GND")
 	)
-	(via
-		(at 130 70)
-		(size 0.6)
-		(drill 0.3)
-		(layers "F.Cu" "B.Cu")
-		(net "GND")
-	)
-	(via
-		(at 150 60)
-		(size 0.6)
-		(drill 0.3)
-		(layers "F.Cu" "B.Cu")
-		(net "GND")
-	)
 	(segment
 		(start 65.734685 67.25)
@@
 	)
 	(segment
-		(start 86 80.4125)
-		(end 79.25 80.4125)
+		(start 79.25 80.4125)
+		(end 79.0875 80.25)
 		(width 0.3)
 		(layer "F.Cu")
@@
 	)
 	(segment
-		(start 86.25 80.6625)
-		(end 86 80.4125)
+		(start 86.25 80.9125)
+		(end 85.75 80.4125)
 		(width 0.3)
 		(layer "F.Cu")
@@
 	)
 	(segment
-		(start 86.25 80.9125)
-		(end 86.25 80.6625)
-		(width 0.3)
-		(layer "F.Cu")
-		(net "Net-(Q1-Pad1)")
-	)
-	(segment
 		(start 75.2025 80.4125)
 		(end 75.04 80.25)
@@
 	)
 	(segment
-		(start 79.25 80.4125)
-		(end 79.0875 80.25)
+		(start 85.75 80.4125)
+		(end 79.25 80.4125)
 		(width 0.3)
 		(layer "F.Cu")
@@
 		)
 	)
-	(group "VIA_STITCHING_GROUPstitch_zone_0"
-		(members "2500ec91-bbdc-4abf-ae23-0441b4b6c331" "5308de85-ea07-427c-a2da-8bde33a71b54"
-			"5655681b-509c-45f3-9d5e-21ef955237da" "64ab616e-88e4-4eca-8c4f-7c67e0d2e65a"
-			"736d4294-3661-4b5e-9a13-ff34b474377e" "9a903746-7582-4a8e-80dc-1afa073be151"
-			"af8a239d-8f5c-44c9-82cb-bb1c3c112a59" "bdb446a1-4f2c-4387-9f77-6333bc5a67b9"
-		)
-	)
-	(group "VIA_STITCHING_GROUP"
-		(members "5db78b2d-af1c-482e-b821-120b0599bb5f" "8ee117d6-1c9f-4a38-96bf-777df4af5a4d"
-			"ff1f01c0-8480-4235-a01c-317088862748"
-		)
-	)
